File: Hardware/LilyPad_XBee.brd (EAGLE design)
At the start: 50 x 50 mm, 40 parts, among them U1 XBEE-1B3, U2 V_REG_LDOSMD

Commit message: Added fiducials
Parts:
- added FID1, FID2: FIDUCIAL1X2, SparkFun-Aesthetics:FIDUCIAL-1X2
